File: LM399_reference_board/LM399_reference_board.sch (EAGLE design)
At the start: 4 parts

Commit message: * Additional work with LM399
Parts:
- added C2: 100n, SquantorRCL:C-EUC0603
- added C3: 10u, SquantorRCL:CPOL-EUSMCD
- added R3: 220k, SquantorRCL:R-EU_0207/10
- added R4: 5k, SquantorRCL:R-EU_0207/10
- added R5: 8.8k, SquantorRCL:R-EU_0207/10
- added R6: 19k, SquantorRCL:R-EU_0207/10
- added R7: (no value), SquantorRCL:R-TRIMMT93YA
- added U$3: LTC2057, SquantorLinearTechnology:LTC2057
- R1, R2: value (none) -> inrush
Connections:
- new net N$6: R5.1, R6.2, U$3.-IN@2, U$3.GRD@1, U$3.GRD@4
- new net N$7: R4.1, R5.2, U$3.OUT@6
- new net N$8: R6.1, R7.A
- new net VZENER: R3.1, R4.2, U$2.C, U$3.+IN@3
- net +15V: now also C2.2, C3.+, R3.2, U$3.V+@8
- net GND: now also C2.1, C3.-, R7.E, R7.S, U$3.V-@5
Changed lines of the file:
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@@
 <part name="C1" library="SquantorRCL" deviceset="CPOL-EU" device="SMCD" value="10u"/>
 <part name="GND3" library="supply1" deviceset="GND" device=""/>
-<part name="R1" library="SquantorRCL" deviceset="R-EU_" device="R1206"/>
-<part name="R2" library="SquantorRCL" deviceset="R-EU_" device="0309/12"/>
+<part name="R1" library="SquantorRCL" deviceset="R-EU_" device="R1206" value="inrush"/>
+<part name="R2" library="SquantorRCL" deviceset="R-EU_" device="0309/12" value="inrush"/>
 <part name="P+1" library="supply1" deviceset="+15V" device=""/>
+<part name="U$3" library="SquantorLinearTechnology" deviceset="LTC2057" device=""/>
+<part name="R3" library="SquantorRCL" deviceset="R-EU_" device="0207/10" value="220k"/>
+<part name="R4" library="SquantorRCL" deviceset="R-EU_" device="0207/10" value="5k"/>
+<part name="R5" library="SquantorRCL" deviceset="R-EU_" device="0207/10" value="8.8k"/>
+<part name="R6" library="SquantorRCL" deviceset="R-EU_" device="0207/10" value="19k"/>
+<part name="GND4" library="supply1" deviceset="GND" device=""/>
+<part name="GND5" library="supply1" deviceset="GND" device=""/>
+<part name="R7" library="SquantorRCL" deviceset="R-TRIMM" device="T93YA"/>
+<part name="P+2" library="supply1" deviceset="+15V" device=""/>
+<part name="GND6" library="supply1" deviceset="GND" device=""/>
+<part name="P+3" library="supply1" deviceset="+15V" device=""/>
+<part name="C2" library="SquantorRCL" deviceset="C-EU" device="C0603" value="100n"/>
+<part name="C3" library="SquantorRCL" deviceset="CPOL-EU" device="SMCD" value="10u"/>
+<part name="P+4" library="supply1" deviceset="+15V" device=""/>
+<part name="GND7" library="supply1" deviceset="GND" device=""/>
 </parts>
 <sheets>
@@
 <instance part="R2" gate="G$1" x="43.18" y="71.12" rot="R90"/>
 <instance part="P+1" gate="1" x="50.8" y="83.82"/>
+<instance part="U$3" gate="G$1" x="121.92" y="58.42"/>
+<instance part="R3" gate="G$1" x="68.58" y="71.12" rot="R90"/>
+<instance part="R4" gate="G$1" x="119.38" y="81.28" rot="R180"/>
+<instance part="R5" gate="G$1" x="119.38" y="76.2"/>
+<instance part="R6" gate="G$1" x="96.52" y="50.8" rot="R90"/>
+<instance part="GND4" gate="1" x="96.52" y="25.4"/>
+<instance part="GND5" gate="1" x="101.6" y="53.34" rot="R270"/>
+<instance part="R7" gate="G$1" x="96.52" y="38.1"/>
+<instance part="P+2" gate="1" x="152.4" y="58.42" rot="R270"/>
+<instance part="GND6" gate="1" x="109.22" y="40.64" rot="R270"/>
+<instance part="P+3" gate="1" x="132.08" y="40.64" rot="R270"/>
+<instance part="C2" gate="G$1" x="119.38" y="40.64" rot="R90"/>
+<instance part="C3" gate="G$1" x="121.92" y="33.02" rot="R270"/>
+<instance part="P+4" gate="1" x="132.08" y="33.02" rot="R270"/>
+<instance part="GND7" gate="1" x="109.22" y="33.02" rot="R270"/>
 </instances>
 <busses>
@@
 <pinref part="GND3" gate="1" pin="GND"/>
 <wire x1="43.18" y1="27.94" x2="43.18" y2="35.56" width="0.1524" layer="91"/>
+</segment>
+<segment>
+<pinref part="U$3" gate="G$1" pin="V-@5"/>
+<pinref part="GND5" gate="1" pin="GND"/>
+</segment>
+<segment>
+<pinref part="GND4" gate="1" pin="GND"/>
+<pinref part="R7" gate="G$1" pin="E"/>
+<wire x1="96.52" y1="33.02" x2="96.52" y2="30.48" width="0.1524" layer="91"/>
+<pinref part="R7" gate="G$1" pin="S"/>
+<wire x1="96.52" y1="30.48" x2="96.52" y2="27.94" width="0.1524" layer="91"/>
+<wire x1="101.6" y1="38.1" x2="104.14" y2="38.1" width="0.1524" layer="91"/>
+<wire x1="104.14" y1="38.1" x2="104.14" y2="30.48" width="0.1524" layer="91"/>
+<wire x1="104.14" y1="30.48" x2="96.52" y2="30.48" width="0.1524" layer="91"/>
+<junction x="96.52" y="30.48"/>
+</segment>
+<segment>
+<pinref part="GND6" gate="1" pin="GND"/>
+<pinref part="C2" gate="G$1" pin="1"/>
+<wire x1="111.76" y1="40.64" x2="116.84" y2="40.64" width="0.1524" layer="91"/>
+</segment>
+<segment>
+<pinref part="GND7" gate="1" pin="GND"/>
+<pinref part="C3" gate="G$1" pin="-"/>
+<wire x1="111.76" y1="33.02" x2="116.84" y2="33.02" width="0.1524" layer="91"/>
 </segment>
 </net>
@@
 <pinref part="P+1" gate="1" pin="+15V"/>
 <wire x1="50.8" y1="78.74" x2="50.8" y2="81.28" width="0.1524" layer="91"/>
+<wire x1="58.42" y1="78.74" x2="68.58" y2="78.74" width="0.1524" layer="91"/>
+<pinref part="R3" gate="G$1" pin="2"/>
+<wire x1="68.58" y1="78.74" x2="68.58" y2="76.2" width="0.1524" layer="91"/>
+<junction x="58.42" y="78.74"/>
+</segment>
+<segment>
+<pinref part="U$3" gate="G$1" pin="V+@8"/>
+<pinref part="P+2" gate="1" pin="+15V"/>
+<wire x1="139.7" y1="58.42" x2="149.86" y2="58.42" width="0.1524" layer="91"/>
+</segment>
+<segment>
+<pinref part="C2" gate="G$1" pin="2"/>
+<pinref part="P+3" gate="1" pin="+15V"/>
+<wire x1="124.46" y1="40.64" x2="129.54" y2="40.64" width="0.1524" layer="91"/>
+</segment>
+<segment>
+<pinref part="C3" gate="G$1" pin="+"/>
+<pinref part="P+4" gate="1" pin="+15V"/>
+<wire x1="124.46" y1="33.02" x2="129.54" y2="33.02" width="0.1524" layer="91"/>
 </segment>
 </net>
+<net name="VZENER" class="0">
+<segment>
+<pinref part="R3" gate="G$1" pin="1"/>
+<wire x1="68.58" y1="66.04" x2="68.58" y2="60.96" width="0.1524" layer="91"/>
+<pinref part="U$2" gate="G$1" pin="C"/>
+<label x="68.58" y="63.5" size="1.778" layer="95"/>
+<pinref part="U$3" gate="G$1" pin="+IN@3"/>
+<wire x1="68.58" y1="60.96" x2="68.58" y2="58.42" width="0.1524" layer="91"/>
+<wire x1="104.14" y1="58.42" x2="88.9" y2="58.42" width="0.1524" layer="91"/>
+<wire x1="88.9" y1="58.42" x2="83.82" y2="58.42" width="0.1524" layer="91"/>
+<wire x1="83.82" y1="58.42" x2="83.82" y2="60.96" width="0.1524" layer="91"/>
+<wire x1="83.82" y1="60.96" x2="68.58" y2="60.96" width="0.1524" layer="91"/>
+<junction x="68.58" y="60.96"/>
+<pinref part="R4" gate="G$1" pin="2"/>
+<wire x1="114.3" y1="81.28" x2="88.9" y2="81.28" width="0.1524" layer="91"/>
+<wire x1="88.9" y1="81.28" x2="88.9" y2="58.42" width="0.1524" layer="91"/>
+<junction x="88.9" y="58.42"/>
+</segment>
+</net>
+<net name="N$7" class="0">
+<segment>
+<pinref part="U$3" gate="G$1" pin="OUT@6"/>
+<wire x1="139.7" y1="53.34" x2="142.24" y2="53.34" width="0.1524" layer="91"/>
+<wire x1="142.24" y1="53.34" x2="142.24" y2="76.2" width="0.1524" layer="91"/>
+<pinref part="R5" gate="G$1" pin="2"/>
+<wire x1="142.24" y1="76.2" x2="129.54" y2="76.2" width="0.1524" layer="91"/>
+<wire x1="129.54" y1="76.2" x2="124.46" y2="76.2" width="0.1524" layer="91"/>
+<wire x1="129.54" y1="76.2" x2="129.54" y2="81.28" width="0.1524" layer="91"/>
+<pinref part="R4" gate="G$1" pin="1"/>
+<wire x1="129.54" y1="81.28" x2="124.46" y2="81.28" width="0.1524" layer="91"/>
+<junction x="129.54" y="76.2"/>
+</segment>
+</net>
+<net name="N$6" class="0">
+<segment>
+<pinref part="R5" gate="G$1" pin="1"/>
+<wire x1="114.3" y1="76.2" x2="96.52" y2="76.2" width="0.1524" layer="91"/>
+<pinref part="R6" gate="G$1" pin="2"/>
+<wire x1="96.52" y1="76.2" x2="96.52" y2="63.5" width="0.1524" layer="91"/>
+<pinref part="U$3" gate="G$1" pin="-IN@2"/>
+<wire x1="96.52" y1="63.5" x2="96.52" y2="60.96" width="0.1524" layer="91"/>
+<wire x1="96.52" y1="60.96" x2="96.52" y2="55.88" width="0.1524" layer="91"/>
+<wire x1="104.14" y1="60.96" x2="96.52" y2="60.96" width="0.1524" layer="91"/>
+<junction x="96.52" y="60.96"/>
+<pinref part="U$3" gate="G$1" pin="GRD@1"/>
+<wire x1="104.14" y1="63.5" x2="96.52" y2="63.5" width="0.1524" layer="91"/>
+<pinref part="U$3" gate="G$1" pin="GRD@4"/>
+<wire x1="104.14" y1="55.88" x2="96.52" y2="55.88" width="0.1524" layer="91"/>
+<junction x="96.52" y="55.88"/>
+<junction x="96.52" y="63.5"/>
+</segment>
+</net>
+<net name="N$8" class="0">
+<segment>
+<pinref part="R6" gate="G$1" pin="1"/>
+<pinref part="R7" gate="G$1" pin="A"/>
+<wire x1="96.52" y1="45.72" x2="96.52" y2="43.18" width="0.1524" layer="91"/>
+</segment>
+</net>
