File: Fluke845_refboard/fluke845_refboard.sch (EAGLE design)
At the start: 0 parts

Commit message: * layed out fluke845 reference board
Parts:
- added C1: 10u, SquantorRCL:C-EUC0805
- added JP1, JP2: (no value), SquantorConnectors:PINHD-1X3TH_SMALL
- added LOGO1: OSHW_LOGO_8MILX0200-NT, ohw-logo:OSHW_LOGO_8MILX0200-NT
- added R1, R2: 33k, SquantorRCL:R-EU_0207/7
- added R3, R4: CALCULATE, SquantorRCL:R-EU_0207/7
- added U$1: SUPERTRONIC37_51, SquantorPCBOutline:SUPERTRONIC37_51
- added U$2, U$3: LT1004, SquantorLinearTechnology:LT1004
Connections:
- new net +15V: JP1.1, R1.2
- new net -15V: JP1.3, R2.1
- new net GND: JP1.2, JP2.2, U$2.A, U$3.C
- new net N$1: C1.2, R2.2, R4.2, U$3.A
- new net N$2: C1.1, R1.1, R3.1, U$2.C
- new net VREF+: JP2.1, R3.2
- new net VREF-: JP2.3, R4.1
