File: PB1_PSU/PB1_PSU.sch (EAGLE design)
At the start: 0 parts

Commit message: * started on the PB1 powersupply
Parts:
- added C1: (no value), SquantorRCL:C-EUC0805
- added C2: (no value), SquantorRCL:CPOL-EUE2.5-7
- added C3: (no value), SquantorRCL:CPOL-EUE5-10.5
- added JP1: POWER_JACKPTH_LOCK, SquantorConnectors:POWER_JACKPTH_LOCK
- added LOGO1: OSHW_LOGO_8MILX0200-NT, ohw-logo:OSHW_LOGO_8MILX0200-NT
- added R1: (no value), SquantorRCL:R-EU_R0805
- added U$1: FUTURLEC_PB1PB1_HALF, SquantorPCBOutline:FUTURLEC_PB1PB1_HALF
- added U$2: BRIDGE_RECTIFIERABS, SquantorDiodes:BRIDGE_RECTIFIERABS
Connections:
- new net AC_EDGE: JP1.GND, R1.1, U$2.AC@2
- new net AC_PIN: JP1.PWR, U$2.AC@1
- new net AC_SW: JP1.GNDBREAK
- new net GND: C1.1, C2.-, C3.-, R1.2, U$2.-
- new net VRECT: C1.2, C2.+, C3.+, U$2.+
