File: PB1_LTC2400_DAQ/PB1_LTC2400_DAQ.sch (EAGLE design)
At the start: 0 parts

Commit message: * updated PB1 board, need a lot more lessons learned with it, so lets leave it for now * updated LTC2400 test board, going to focus on that first
Parts:
- added C1, C10, C12, C2, C7, C9: 100n, SquantorRCL:C-EUC1812K
- added C11, C8: 100n, SquantorRCL:C-EUC0603
- added C13: (no value), SquantorRCL:C-EU075-063X106
- added C3, C4, C5, C6: 1u, SquantorRCL:C-EUC2220K
- added LOGO1: OSHW_LOGO_8MILX0200-NT, ohw-logo:OSHW_LOGO_8MILX0200-NT
- added R1, R2: 0, SquantorRCL:R-EU_R0805
- added R3, R5: 1k, SquantorRCL:R-EU_R0805
- added R4: 20k, SquantorRCL:R-EU_R0805
- added U$1: FUTURLEC_PB1PB1, SquantorPCBOutline:FUTURLEC_PB1PB1
- added U$2: LTC6655LS8_ELONG, SquantorLinearTechnology:LTC6655LS8_ELONG
- added U$3, U$4: LTC2057, SquantorLinearTechnology:LTC2057
- added U1: LTC2400CS8PBF, SquantorLinearTechnology:LTC2400CS8PBF
- added U2: LTC1043CSWPBFSW, SquantorLinearTechnology:LTC1043CSWPBFSW
- added X1: (no value), con-subd:F09VP
Connections:
- new net +5V: C1.1, C10.1, C12.1, C9.1, U$2./SHDN@1, U$2.VIN@2, U$3.V+@8, U$4.V+@8, U1.VCC, U2.V+
- new net -5V: C10.2, C2.1, C7.2, C9.2, U$3.V-@5, U$4.V-@5, U2.V-
- new net CA+: C3.1, U2.CA+
- new net CA-: C3.2, U2.CA-
- new net CA_GUARD: U2.SHA
- new net CB+: C4.1, U2.CB+
- new net CB-: C4.2, U2.CB-
- new net CB_GUARD: U2.SHB
- new net COSC: C7.1, U2.COSC
- new net DIFF_IN_1: U2.S1A
- new net DIFF_IN_2: U2.S3A
- new net GND: C1.2, C12.2, C13.1, C2.2, C5.2, U$2.GND@3, U$2.GND@4, U$2.GND@5, U$2.GND@8, U1.GND, U2.S4B
- new net N$1: R5.2, U1.VIN
- new net N$2: U$4.GRD@4
- new net N$5: U$4.GRD@1
- new net OUT_AMP: R4.2, R5.1, U$4.OUT@6
- new net OUT_BUF: R2.2, R3.1, U$3.OUT@6
- new net SDCOM_AMP: C8.2, U$4.SDCOM@9
- new net SDCOM_BUF: C11.2, U$3.SDCOM@9
- new net SD_AMP: C8.1, U$4./SD@10
- new net SD_BUF: C11.1, U$3./SD@10
- new net V+_AMP: U$4.+IN@3
- new net V+_BUF: R1.2, U$3.+IN@3
- new net V-_AMP: R3.2, R4.1, U$4.-IN@2
- new net V-_BUF: R2.1, U$3.-IN@2, U$3.GRD@4
- new net VOUT: C6.1, U2.S2A
- new net VREF: C13.2, U$2.VOUT_F@7, U$2.VOUT_S@6, U1.VREF, U2.S1B
- new net VREF/2: C5.1, C6.2, R1.1, U2.S2B, U2.S3B, U2.S4A
