File: adc_modules/ltc2400_adc_module.sch (EAGLE design)
At the start: 0 parts

Commit message: * small modifications on ltc2400_adc_module
Parts:
- added C3: 10u, SquantorRCL:C-EUC0805
- added JP1, JP2: (no value), SquantorConnectors:PINHD-1X10NORM_OCT
- added R2: ferrite, SquantorRCL:R-EU_R0805
Connections:
- new net GND: C3.1, JP1.2, JP1.3, JP1.6, JP2.1, JP2.2
- new net GND_ADC: JP2.9
- new net N$1: JP1.1, R2.1
- new net N$13: JP2.3
- new net N$14: JP2.4
- new net N$15: JP2.5
- new net N$16: JP2.6
- new net N$17: JP2.7
- new net N$18: JP2.8
- new net V+: JP1.7
- new net V-: JP1.10
- new net VCC_ADC: JP2.10
- new net VCC_VREF: C3.2, R2.2
- new net VIN+: JP1.8
- new net VIN-: JP1.9
- new net VREF_IN: JP1.4
- new net VREF_OUT: JP1.5
