File: adc_modules/mcp3551_adc_module.sch (EAGLE design)
At the start: 0 parts

Commit message: * updated and almost finished MCP3551 ADC module
Parts:
- added C1: 100n, SquantorRCL:C-EUC0603
- added C3: 10u, SquantorRCL:C-EUC0805
- added R1, R3, R4: 100, SquantorRCL:R-EU_R0603
- added R2: ferrite, SquantorRCL:R-EU_R0805
- added R5, R6: 5.1k, SquantorRCL:R-EU_R0805
- added U$1: METROLOGY_MODULE1.5MM, SquantorPCBOutline:METROLOGY_MODULE1.5MM
- added U1: MCP3553-E/SN, SquantorMicrochip:MCP3553-E/SN
Connections:
- new net ADC_CS: R1.1, U1.CS*
- new net ADC_SCK: R4.1, U1.SCK
- new net ADC_SDO: R3.1, U1.SDO/RDY*
- new net ADC_VIN+: R5.1, U1.VIN+
- new net ADC_VIN-: R6.1, U1.VIN-
- new net GND: C1.1, C3.1, U$1.GND_ADC@19, U$1.GND_VREF@6, U$1.V-@10, U1.VSS
- new net N$1: R2.1, U$1.VCC_ADC@20
- new net N$2: R1.2, U$1.ADC_CTRL@18
- new net N$3: R3.2, U$1.ADC_CTRL@17
- new net N$4: R4.2, U$1.ADC_CTRL@16
- new net N$5: R5.2, U$1.VIN+@8
- new net N$6: R6.2, U$1.VIN-@9
- new net VCC: C1.2, C3.2, R2.2, U1.VDD
- new net VREF: U$1.V+@7, U$1.VREF_IN@4, U$1.VREF_OUT@5, U1.VREF
