File: reference_modules/lt1236LS8_reference_module.sch (EAGLE design)
At the start: 0 parts

Commit message: * modified boards and processed for production
Parts:
- added C1, C6: 100n, SquantorRCL:C-EUC0603
- added C2, C4, C5: 1u, SquantorRCL:C-EU025-060X050
- added C3: 10u, SquantorRCL:C-EUC0805
- added NTC, RTRIM: (no value), SquantorRCL:R-EU_R0805
- added R1: 27k, SquantorRCL:R-EU_R0805
- added R2: ferrite, SquantorRCL:R-EU_R0805
- added R3: 50k, SquantorRCL:R-TRIMM3224W
- added R4, R5: 36k, SquantorRCL:R-EU_R0805
- added U$1: LT1001, SquantorLinearTechnology:LT1001
- added U$2: METROLOGY_MODULE, SquantorPCBOutline:METROLOGY_MODULE
- added U$3: BAS17, SquantorNxp:BAS17
- added U1: LT1236BILS8-5PBFLS8_ELONG, SquantorLinearTechnology:LT1236BILS8-5PBFLS8_ELONG
Connections:
- new net GND: C1.2, C3.1, C5.2, C6.2, NTC.1, R3.E, U$1.V-, U$2.GND_VREF@2, U$2.GND_VREF@3, U$2.GND_VREF@6, U1.GND@4
- new net N$1: R2.1, U$2.VCC_VREF@1
- new net N$2: R3.S, RTRIM.2, U$3.C
- new net N$3: NTC.2, RTRIM.1
- new net N$5: C2.1, R4.1, R5.2
- new net N$6: C4.1, R4.2, U$1.+IN
- new net N$8: C4.2, C5.1
- new net VCC_VREF: C1.1, C3.2, C6.1, R2.2, U$1.V+, U1.VIN@2
- new net VREF_IN: C2.2, U$1.-IN, U$2.VREF_IN@4
- new net VREF_OUT: U$1.OUT, U$2.VREF_OUT@5
- new net VREF_OUT_UNFILT: R1.2, R3.A, R5.1, U1.VOUT@6
- new net VREF_TRIM: R1.1, U$3.A, U1.TRIM@5
