File: kicad/MCP355X_module/MCP355X_module.sch (KiCad schematic (older format))
At the start: 16 parts, among them J1 PINS_1X8, J2 PINS_1X8, U1 MCP355X-E_SN

Commit message: * finished routing MCP355X PCB
Parts:
- removed J1, J2: PINS_1X8, SquantorConnectors:Header-2.54-1X08-H1.5, symbol PINS_1X8
- added C1: 1u, Capacitors_SMD:C_0805, symbol C
- added C2: 10n, Capacitors_SMD:C_0603, symbol C
- added J1, J2: PINS_1X6, SquantorConnectors:Header-2.54-1X06-H1.5, symbol PINS_1X6
- added R1: 100, Resistors_SMD:R_0603, symbol R
- C4, C8: footprint SquantorRcl:SquantorRCL-C025-050X050 -> SquantorRcl:RCL-C025-050X050
- C9: footprint SquantorRcl:SquantorRCL-C025-025X050 -> Capacitors_SMD:C_0603
Connections:
- wire segments 40 -> 42
Changed lines of the file:
@@
 	1    0    0    -1
 $EndComp
-Wire Wire Line
-	2050 2600 2150 2600
 $Comp
 L GND #PWR01
@@
 L VDD #PWR03
 U 1 1 584C1814
-P 5450 2100
-F 0 "#PWR03" H 5450 1950 50  0001 C CNN
-F 1 "VDD" H 5450 2250 50  0000 C CNN
-F 2 "" H 5450 2100 50  0000 C CNN
-F 3 "" H 5450 2100 50  0000 C CNN
-	1    5450 2100
+P 5100 2100
+F 0 "#PWR03" H 5100 1950 50  0001 C CNN
+F 1 "VDD" H 5100 2250 50  0000 C CNN
+F 2 "" H 5100 2100 50  0000 C CNN
+F 3 "" H 5100 2100 50  0000 C CNN
+	1    5100 2100
 	0    -1   -1   0
 $EndComp
@@
 F 0 "C4" H 2825 1950 50  0000 L CNN
 F 1 "1u" H 2825 1750 50  0000 L CNN
-F 2 "SquantorRcl:SquantorRCL-C025-050X050" H 2800 2400 50  0001 C CNN
+F 2 "SquantorRcl:RCL-C025-050X050" H 2800 2400 50  0001 C CNN
 F 3 "" H 2800 1850 50  0000 C CNN
 	1    2800 1850
@@
 F 0 "C8" H 3275 1950 50  0000 L CNN
 F 1 "1u" H 3275 1750 50  0000 L CNN
-F 2 "SquantorRcl:SquantorRCL-C025-050X050" H 3250 2300 50  0001 C CNN
+F 2 "SquantorRcl:RCL-C025-050X050" H 3250 2300 50  0001 C CNN
 F 3 "" H 3250 1850 50  0000 C CNN
 	1    3250 1850
@@
 Connection ~ 2800 2100
 $Comp
-L GND #PWR05
+L GND #PWR04
 U 1 1 584C2957
 P 2800 1650
-F 0 "#PWR05" H 2800 1400 50  0001 C CNN
+F 0 "#PWR04" H 2800 1400 50  0001 C CNN
 F 1 "GND" H 2800 1500 50  0000 C CNN
 F 2 "" H 2800 1650 50  0000 C CNN
@@
 $EndComp
 $Comp
-L GND #PWR06
+L GND #PWR05
 U 1 1 584C2980
 P 3250 1650
-F 0 "#PWR06" H 3250 1400 50  0001 C CNN
+F 0 "#PWR05" H 3250 1400 50  0001 C CNN
 F 1 "GND" H 3250 1500 50  0000 C CNN
 F 2 "" H 3250 1650 50  0000 C CNN
@@
 F 0 "C9" H 3575 1950 50  0000 L CNN
 F 1 "10n" H 3575 1750 50  0000 L CNN
-F 2 "SquantorRcl:SquantorRCL-C025-025X050" H 3588 1700 50  0000 C CNN
+F 2 "Capacitors_SMD:C_0603" H 3588 1700 50  0001 C CNN
 F 3 "" H 3550 1850 50  0000 C CNN
 	1    3550 1850
@@
 	2800 1650 2800 1700
 $Comp
-L GND #PWR07
+L GND #PWR06
 U 1 1 584C272D
 P 3550 1650
-F 0 "#PWR07" H 3550 1400 50  0001 C CNN
+F 0 "#PWR06" H 3550 1400 50  0001 C CNN
 F 1 "GND" H 3550 1500 50  0000 C CNN
 F 2 "" H 3550 1650 50  0000 C CNN
@@
 $EndComp
 $Comp
-L GND #PWR08
+L GND #PWR07
 U 1 1 584C2F9D
 P 3000 3550
-F 0 "#PWR08" H 3000 3300 50  0001 C CNN
+F 0 "#PWR07" H 3000 3300 50  0001 C CNN
 F 1 "GND" H 3000 3400 50  0000 C CNN
 F 2 "" H 3000 3550 50  0000 C CNN
@@
 $EndComp
 $Comp
-L GND #PWR011
+L GND #PWR08
 U 1 1 584C307B
 P 3000 2350
-F 0 "#PWR011" H 3000 2100 50  0001 C CNN
+F 0 "#PWR08" H 3000 2100 50  0001 C CNN
 F 1 "GND" H 3000 2200 50  0000 C CNN
 F 2 "" H 3000 2350 50  0000 C CNN
@@
 	3000 3550 3000 3500
 Wire Wire Line
-	2100 2500 2050 2500
-Wire Wire Line
-	2100 2500 2100 2700
-Connection ~ 2100 2600
-$Comp
-L GND #PWR012
+	2050 2500 2150 2500
+$Comp
+L GND #PWR09
 U 1 1 584C38A2
-P 2150 2600
-F 0 "#PWR012" H 2150 2350 50  0001 C CNN
-F 1 "GND" H 2150 2450 50  0000 C CNN
-F 2 "" H 2150 2600 50  0000 C CNN
-F 3 "" H 2150 2600 50  0000 C CNN
-	1    2150 2600
+P 2150 2500
+F 0 "#PWR09" H 2150 2250 50  0001 C CNN
+F 1 "GND" H 2150 2350 50  0000 C CNN
+F 2 "" H 2150 2500 50  0000 C CNN
+F 3 "" H 2150 2500 50  0000 C CNN
+	1    2150 2500
 	0    -1   -1   0
 $EndComp
@@
 	3350 3150 3350 2300
 $Comp
-L PINS_1X8 J1
-U 1 1 584C4620
-P 1850 2350
-F 0 "J1" H 1800 2850 60  0000 C CNN
-F 1 "PINS_1X8" H 1850 1850 60  0000 C CNN
-F 2 "SquantorConnectors:Header-2.54-1X08-H1.5" H 1850 2700 60  0001 C CNN
-F 3 "" H 1850 2700 60  0001 C CNN
-	1    1850 2350
-	1    0    0    -1
-$EndComp
-$Comp
-L PINS_1X8 J2
-U 1 1 584C4743
-P 5700 2250
-F 0 "J2" H 5650 2750 60  0000 C CNN
-F 1 "PINS_1X8" H 5700 1750 60  0000 C CNN
-F 2 "SquantorConnectors:Header-2.54-1X08-H1.5" H 5700 2600 60  0001 C CNN
-F 3 "" H 5700 2600 60  0001 C CNN
-	1    5700 2250
-	-1   0    0    1
-$EndComp
-$Comp
-L GND #PWR?
+L GND #PWR010
 U 1 1 584C4B15
 P 2100 2000
-F 0 "#PWR?" H 2100 1750 50  0001 C CNN
+F 0 "#PWR010" H 2100 1750 50  0001 C CNN
 F 1 "GND" H 2100 1850 50  0000 C CNN
 F 2 "" H 2100 2000 50  0000 C CNN
@@
 	2050 2000 2100 2000
 $Comp
-L GND #PWR?
+L GND #PWR011
 U 1 1 584C4C15
 P 2100 2200
-F 0 "#PWR?" H 2100 1950 50  0001 C CNN
+F 0 "#PWR011" H 2100 1950 50  0001 C CNN
 F 1 "GND" H 2100 2050 50  0000 C CNN
 F 2 "" H 2100 2200 50  0000 C CNN
@@
 Wire Wire Line
 	2400 2400 2050 2400
-Wire Wire Line
-	2100 2700 2050 2700
+$Comp
+L C C2
+U 1 1 584C446E
+P 4500 1800
+F 0 "C2" H 4525 1900 50  0000 L CNN
+F 1 "10n" H 4525 1700 50  0000 L CNN
+F 2 "Capacitors_SMD:C_0603" H 4538 1650 50  0001 C CNN
+F 3 "" H 4500 1800 50  0000 C CNN
+	1    4500 1800
+	0    1    1    0
+$EndComp
+$Comp
+L C C1
+U 1 1 584C4507
+P 4500 1550
+F 0 "C1" H 4525 1650 50  0000 L CNN
+F 1 "1u" H 4525 1450 50  0000 L CNN
+F 2 "Capacitors_SMD:C_0805" H 4538 1400 50  0001 C CNN
+F 3 "" H 4500 1550 50  0000 C CNN
+	1    4500 1550
+	0    1    1    0
+$EndComp
+$Comp
+L VDD #PWR012
+U 1 1 584C45EC
+P 4700 1800
+F 0 "#PWR012" H 4700 1650 50  0001 C CNN
+F 1 "VDD" H 4700 1950 50  0000 C CNN
+F 2 "" H 4700 1800 50  0000 C CNN
+F 3 "" H 4700 1800 50  0000 C CNN
+	1    4700 1800
+	0    1    1    0
+$EndComp
+$Comp
+L VDD #PWR013
+U 1 1 584C468E
+P 4700 1550
+F 0 "#PWR013" H 4700 1400 50  0001 C CNN
+F 1 "VDD" H 4700 1700 50  0000 C CNN
+F 2 "" H 4700 1550 50  0000 C CNN
+F 3 "" H 4700 1550 50  0000 C CNN
+	1    4700 1550
+	0    1    1    0
+$EndComp
+$Comp
+L GND #PWR014
+U 1 1 584C46CF
+P 4300 1800
+F 0 "#PWR014" H 4300 1550 50  0001 C CNN
+F 1 "GND" H 4300 1650 50  0000 C CNN
+F 2 "" H 4300 1800 50  0000 C CNN
+F 3 "" H 4300 1800 50  0000 C CNN
+	1    4300 1800
+	0    1    1    0
+$EndComp
+$Comp
+L GND #PWR015
+U 1 1 584C4710
+P 4300 1550
+F 0 "#PWR015" H 4300 1300 50  0001 C CNN
+F 1 "GND" H 4300 1400 50  0000 C CNN
+F 2 "" H 4300 1550 50  0000 C CNN
+F 3 "" H 4300 1550 50  0000 C CNN
+	1    4300 1550
+	0    1    1    0
+$EndComp
+Wire Wire Line
+	4700 1800 4650 1800
+Wire Wire Line
+	4700 1550 4650 1550
+Wire Wire Line
+	4300 1550 4350 1550
+Wire Wire Line
+	4300 1800 4350 1800
+$Comp
+L R R1
+U 1 1 584C4B10
+P 5300 2100
+F 0 "R1" V 5380 2100 50  0000 C CNN
+F 1 "100" V 5300 2100 50  0000 C CNN
+F 2 "Resistors_SMD:R_0603" V 5650 2200 50  0001 C CNN
+F 3 "" H 5300 2100 50  0000 C CNN
+	1    5300 2100
+	0    1    1    0
+$EndComp
+Wire Wire Line
+	5150 2100 5100 2100
+$Comp
+L PINS_1X6 J1
+U 1 1 584C58EB
+P 1850 2250
+F 0 "J1" H 1800 2650 60  0000 C CNN
+F 1 "PINS_1X6" H 1850 1850 60  0000 C CNN
+F 2 "SquantorConnectors:Header-2.54-1X06-H1.5" H 1850 2500 60  0001 C CNN
+F 3 "" H 1850 2500 60  0001 C CNN
+	1    1850 2250
+	1    0    0    -1
+$EndComp
+$Comp
+L PINS_1X6 J2
+U 1 1 584C5985
+P 5700 2150
+F 0 "J2" H 5650 2550 60  0000 C CNN
+F 1 "PINS_1X6" H 5700 1750 60  0000 C CNN
+F 2 "SquantorConnectors:Header-2.54-1X06-H1.5" H 5700 2400 60  0001 C CNN
+F 3 "" H 5700 2400 60  0001 C CNN
+	1    5700 2150
+	-1   0    0    1
+$EndComp
 $EndSCHEMATC

Commit message: * small mods and optimizations
Parts:
- J1, J2: footprint SquantorConnectors:Header-2.54-1X06-H1.5 -> SquantorConnectors:Header-2.54-1X06-H0.8
Connections:
- net Vref: now reaches C8.2, C9.2, R6.1, U1.1 (Vref)
- net Vin+filt: now reaches C5.2, C6.1, R4.1, U1.2 (Vin+)
- net Vin-_filt: now reaches C6.2, C7.1, R5.1, U1.3 (Vin-)
- net Vref_filt: now reaches C4.2, R3.1, R6.2
- net Vref_in: now reaches J1.2, R3.2
- net Vin+_in: now reaches J1.4, R4.2
- net Vin-_in: now reaches J1.5, R5.2
Changed lines of the file:
@@
 	3000 3550 3000 3500
 Wire Wire Line
-	2050 2500 2150 2500
+	2050 2500 2100 2500
 $Comp
 L GND #PWR09
 U 1 1 584C38A2
-P 2150 2500
-F 0 "#PWR09" H 2150 2250 50  0001 C CNN
-F 1 "GND" H 2150 2350 50  0000 C CNN
-F 2 "" H 2150 2500 50  0000 C CNN
-F 3 "" H 2150 2500 50  0000 C CNN
-	1    2150 2500
+P 2100 2500
+F 0 "#PWR09" H 2100 2250 50  0001 C CNN
+F 1 "GND" H 2100 2350 50  0000 C CNN
+F 2 "" H 2100 2500 50  0000 C CNN
+F 3 "" H 2100 2500 50  0000 C CNN
+	1    2100 2500
 	0    -1   -1   0
 $EndComp
@@
 	2100 2200 2050 2200
 Wire Wire Line
-	2400 2100 2050 2100
+	2050 2100 2400 2100
 Wire Wire Line
 	2050 2300 2500 2300
@@
 F 0 "J1" H 1800 2650 60  0000 C CNN
 F 1 "PINS_1X6" H 1850 1850 60  0000 C CNN
-F 2 "SquantorConnectors:Header-2.54-1X06-H1.5" H 1850 2500 60  0001 C CNN
+F 2 "SquantorConnectors:Header-2.54-1X06-H0.8" H 1850 2500 60  0001 C CNN
 F 3 "" H 1850 2500 60  0001 C CNN
 	1    1850 2250
@@
 F 0 "J2" H 5650 2550 60  0000 C CNN
 F 1 "PINS_1X6" H 5700 1750 60  0000 C CNN
-F 2 "SquantorConnectors:Header-2.54-1X06-H1.5" H 5700 2400 60  0001 C CNN
+F 2 "SquantorConnectors:Header-2.54-1X06-H0.8" H 5700 2400 60  0001 C CNN
 F 3 "" H 5700 2400 60  0001 C CNN
 	1    5700 2150
 	-1   0    0    1
 $EndComp
+Text Label 2350 2000 0    60   ~ 0
+Vref_in
+Wire Wire Line
+	2350 2000 2350 2100
+Connection ~ 2350 2100
+Text Label 2800 2100 3    60   ~ 0
+Vref_filt
+Text Label 3300 2100 0    60   ~ 0
+Vref
+Text Label 3000 2750 0    60   ~ 0
+Vin+filt
+Text Label 3000 3150 0    60   ~ 0
+Vin-_filt
+Text Label 2500 2600 0    60   ~ 0
+Vin+_in
+Text Label 2400 2950 0    60   ~ 0
+Vin-_in
 $EndSCHEMATC

Commit message: * changed input filter caps from 0603 to 0805
Parts:
- C5, C6, C7: footprint Capacitors_SMD:C_0603 -> Capacitors_SMD:C_0805
Changed lines of the file:
@@
 F 0 "C6" H 3025 3050 50  0000 L CNN
 F 1 "C" H 3025 2850 50  0000 L CNN
-F 2 "Capacitors_SMD:C_0603" H 3038 2800 50  0001 C CNN
+F 2 "Capacitors_SMD:C_0805" H 3038 2800 50  0001 C CNN
 F 3 "" H 3000 2950 50  0000 C CNN
 	1    3000 2950
@@
 F 0 "C5" H 3025 2650 50  0000 L CNN
 F 1 "C" H 3025 2450 50  0000 L CNN
-F 2 "Capacitors_SMD:C_0603" H 3038 2400 50  0001 C CNN
+F 2 "Capacitors_SMD:C_0805" H 3038 2400 50  0001 C CNN
 F 3 "" H 3000 2550 50  0000 C CNN
 	1    3000 2550
@@
 F 0 "C7" H 3025 3450 50  0000 L CNN
 F 1 "C" H 3025 3250 50  0000 L CNN
-F 2 "Capacitors_SMD:C_0603" H 3038 3200 50  0001 C CNN
+F 2 "Capacitors_SMD:C_0805" H 3038 3200 50  0001 C CNN
 F 3 "" H 3000 3350 50  0000 C CNN
 	1    3000 3350

Commit message: * changed bad footprints for the WIMA MKS-02 1uF caps
Parts:
- C4, C8: footprint SquantorRcl:RCL-C025-050X050 -> SquantorRcl:C025-055X046
Changed lines of the file:
@@
 F 0 "C4" H 2825 1950 50  0000 L CNN
 F 1 "1u" H 2825 1750 50  0000 L CNN
-F 2 "SquantorRcl:RCL-C025-050X050" H 2800 2400 50  0001 C CNN
+F 2 "SquantorRcl:C025-055X046" H 2800 2400 50  0001 C CNN
 F 3 "" H 2800 1850 50  0000 C CNN
 	1    2800 1850
@@
 F 0 "C8" H 3275 1950 50  0000 L CNN
 F 1 "1u" H 3275 1750 50  0000 L CNN
-F 2 "SquantorRcl:RCL-C025-050X050" H 3250 2300 50  0001 C CNN
+F 2 "SquantorRcl:C025-055X046" H 3250 2300 50  0001 C CNN
 F 3 "" H 3250 1850 50  0000 C CNN
 	1    3250 1850
