File: kicad/LTC6655_module/LTC6655_module.sch (KiCad schematic (older format))
At the start: 3 parts, among them J1 PINS_1X6, J2 PINS_1X6, M1 LTC6655LS8

Commit message: * updated the LTC6655 reference board
Parts:
- removed J1, J2: PINS_1X6, SquantorConnectors:Header-2.54-1X06-H0.8, symbol PINS_1X6
- added C1: 1u, Capacitors_SMD:C_0603, symbol C
- added C2: 10n, Capacitors_SMD:C_0805, symbol C
- added C3: 6.8u, SquantorRcl:C050-085X075, symbol C
- added J1, J2: PINS_1X8, SquantorConnectors:Header-0254-1X08-H010, symbol PINS_1X8
- added R1: 0, Resistors_SMD:R_0603, symbol R
- M1: footprint SquantorLinearTechnology:SquantorLinearTechnology-LS8 -> SquantorLinearTechnology:LS8_ELONG
Connections:
- net labels added: Heater, HeaterGround, RefTemp, Sense, Vin, Vref
- wire segments 5 -> 43
