File: kicad/REF50XX_module/REF50XX_module.sch (KiCad schematic (older format))
At the start: 3 parts

Commit message: * added REF schematic stuff
Parts:
- added C? (x2): 1u, symbol C
- added C?: C, symbol C
- added C?: 10u, symbol C
- added R?: 470k, symbol R
- added R?: 1k, symbol R
- added R?: 1, symbol R
- added RV?: 10k, symbol POT
Connections:
- wire segments 2 -> 19
Other:
- moved on the sheet: U?
Changed lines of the file:
@@
 LIBS:SquantorConnectors
 LIBS:SquantorTexasInstruments
+LIBS:REF50XX_module-cache
 EELAYER 25 0
 EELAYER END
@@
 L PINS_1X6 J?
 U 1 1 584C8340
-P 3000 1350
-F 0 "J?" H 2950 1750 60  0000 C CNN
-F 1 "PINS_1X6" H 3000 950 60  0000 C CNN
-F 2 "" H 3000 1600 60  0001 C CNN
-F 3 "" H 3000 1600 60  0001 C CNN
-	1    3000 1350
+P 4100 1350
+F 0 "J?" H 4050 1750 60  0000 C CNN
+F 1 "PINS_1X6" H 4100 950 60  0000 C CNN
+F 2 "" H 4100 1600 60  0001 C CNN
+F 3 "" H 4100 1600 60  0001 C CNN
+	1    4100 1350
 	-1   0    0    1
 $EndComp
@@
 L REF50X0 U?
 U 1 1 584C8585
-P 1950 1400
-F 0 "U?" H 1950 1750 60  0000 C CNN
-F 1 "REF50X0" H 1950 1150 60  0000 C CNN
-F 2 "" H 1900 1400 60  0001 C CNN
-F 3 "" H 1900 1400 60  0001 C CNN
-	1    1950 1400
+P 2400 1400
+F 0 "U?" H 2400 1750 60  0000 C CNN
+F 1 "REF50X0" H 2400 1150 60  0000 C CNN
+F 2 "" H 2350 1400 60  0001 C CNN
+F 3 "" H 2350 1400 60  0001 C CNN
+	1    2400 1400
 	1    0    0    -1
 $EndComp
@@
 L GND #PWR?
 U 1 1 584C862D
-P 1500 1500
-F 0 "#PWR?" H 1500 1250 50  0001 C CNN
-F 1 "GND" H 1500 1350 50  0000 C CNN
-F 2 "" H 1500 1500 50  0000 C CNN
-F 3 "" H 1500 1500 50  0000 C CNN
-	1    1500 1500
+P 1950 1500
+F 0 "#PWR?" H 1950 1250 50  0001 C CNN
+F 1 "GND" H 1950 1350 50  0000 C CNN
+F 2 "" H 1950 1500 50  0000 C CNN
+F 3 "" H 1950 1500 50  0000 C CNN
+	1    1950 1500
 	0    1    1    0
 $EndComp
@@
 	1150 1600 1200 1600
 Wire Wire Line
-	1500 1500 1550 1500
+	1950 1500 2000 1500
+$Comp
+L C C?
+U 1 1 58545DF7
+P 2850 1700
+F 0 "C?" H 2875 1800 50  0000 L CNN
+F 1 "1u" H 2875 1600 50  0000 L CNN
+F 2 "" H 2888 1550 50  0000 C CNN
+F 3 "" H 2850 1700 50  0000 C CNN
+	1    2850 1700
+	1    0    0    -1
+$EndComp
+$Comp
+L C C?
+U 1 1 58545FD9
+P 1800 1100
+F 0 "C?" H 1825 1200 50  0000 L CNN
+F 1 "C" H 1825 1000 50  0000 L CNN
+F 2 "" H 1838 950 50  0000 C CNN
+F 3 "" H 1800 1100 50  0000 C CNN
+	1    1800 1100
+	1    0    0    -1
+$EndComp
+$Comp
+L C C?
+U 1 1 5854616F
+P 3200 850
+F 0 "C?" H 3225 950 50  0000 L CNN
+F 1 "10u" H 3225 750 50  0000 L CNN
+F 2 "" H 3238 700 50  0000 C CNN
+F 3 "" H 3200 850 50  0000 C CNN
+	1    3200 850
+	1    0    0    -1
+$EndComp
+$Comp
+L C C?
+U 1 1 585461DE
+P 3450 850
+F 0 "C?" H 3475 950 50  0000 L CNN
+F 1 "1u" H 3475 750 50  0000 L CNN
+F 2 "" H 3488 700 50  0000 C CNN
+F 3 "" H 3450 850 50  0000 C CNN
+	1    3450 850
+	1    0    0    -1
+$EndComp
+$Comp
+L GND #PWR?
+U 1 1 585462A7
+P 2850 1900
+F 0 "#PWR?" H 2850 1650 50  0001 C CNN
+F 1 "GND" H 2850 1750 50  0000 C CNN
+F 2 "" H 2850 1900 50  0000 C CNN
+F 3 "" H 2850 1900 50  0000 C CNN
+	1    2850 1900
+	1    0    0    -1
+$EndComp
+$Comp
+L GND #PWR?
+U 1 1 585462C7
+P 3200 650
+F 0 "#PWR?" H 3200 400 50  0001 C CNN
+F 1 "GND" H 3200 500 50  0000 C CNN
+F 2 "" H 3200 650 50  0000 C CNN
+F 3 "" H 3200 650 50  0000 C CNN
+	1    3200 650
+	-1   0    0    1
+$EndComp
+$Comp
+L GND #PWR?
+U 1 1 58546306
+P 3450 650
+F 0 "#PWR?" H 3450 400 50  0001 C CNN
+F 1 "GND" H 3450 500 50  0000 C CNN
+F 2 "" H 3450 650 50  0000 C CNN
+F 3 "" H 3450 650 50  0000 C CNN
+	1    3450 650
+	-1   0    0    1
+$EndComp
+Wire Wire Line
+	3200 700  3200 650
+Wire Wire Line
+	3450 700  3450 650
+Wire Wire Line
+	3200 1400 3200 1350
+Connection ~ 3200 1400
+$Comp
+L GND #PWR?
+U 1 1 5854639C
+P 1800 900
+F 0 "#PWR?" H 1800 650 50  0001 C CNN
+F 1 "GND" H 1800 750 50  0000 C CNN
+F 2 "" H 1800 900 50  0000 C CNN
+F 3 "" H 1800 900 50  0000 C CNN
+	1    1800 900
+	-1   0    0    1
+$EndComp
+Wire Wire Line
+	1800 950  1800 900
+Wire Wire Line
+	2000 1300 1800 1300
+Wire Wire Line
+	1800 1300 1800 1250
+$Comp
+L R R?
+U 1 1 58546469
+P 3050 1500
+F 0 "R?" V 3130 1500 50  0000 C CNN
+F 1 "470k" V 3050 1500 50  0000 C CNN
+F 2 "" V 2980 1500 50  0000 C CNN
+F 3 "" H 3050 1500 50  0000 C CNN
+	1    3050 1500
+	0    1    1    0
+$EndComp
+$Comp
+L POT RV?
+U 1 1 585464D5
+P 3450 1700
+F 0 "RV?" H 3450 1620 50  0000 C CNN
+F 1 "10k" H 3450 1700 50  0000 C CNN
+F 2 "" H 3450 1700 50  0000 C CNN
+F 3 "" H 3450 1700 50  0000 C CNN
+	1    3450 1700
+	0    -1   -1   0
+$EndComp
+Wire Wire Line
+	2800 1500 2900 1500
+Wire Wire Line
+	2850 1550 2850 1500
+Connection ~ 2850 1500
+Wire Wire Line
+	2850 1900 2850 1850
+Wire Wire Line
+	3200 1500 3250 1500
+Wire Wire Line
+	3250 1500 3250 1700
+Wire Wire Line
+	3250 1700 3300 1700
+Wire Wire Line
+	3450 1000 3450 1550
+Connection ~ 3450 1400
+$Comp
+L R R?
+U 1 1 585467AF
+P 3450 2050
+F 0 "R?" V 3530 2050 50  0000 C CNN
+F 1 "1k" V 3450 2050 50  0000 C CNN
+F 2 "" V 3380 2050 50  0000 C CNN
+F 3 "" H 3450 2050 50  0000 C CNN
+	1    3450 2050
+	1    0    0    -1
+$EndComp
+$Comp
+L GND #PWR?
+U 1 1 5854682E
+P 3450 2250
+F 0 "#PWR?" H 3450 2000 50  0001 C CNN
+F 1 "GND" H 3450 2100 50  0000 C CNN
+F 2 "" H 3450 2250 50  0000 C CNN
+F 3 "" H 3450 2250 50  0000 C CNN
+	1    3450 2250
+	1    0    0    -1
+$EndComp
+Wire Wire Line
+	3450 2250 3450 2200
+Wire Wire Line
+	3450 1900 3450 1850
+$Comp
+L R R?
+U 1 1 58546B54
+P 3200 1200
+F 0 "R?" V 3280 1200 50  0000 C CNN
+F 1 "1" V 3200 1200 50  0000 C CNN
+F 2 "" V 3130 1200 50  0000 C CNN
+F 3 "" H 3200 1200 50  0000 C CNN
+	1    3200 1200
+	1    0    0    -1
+$EndComp
+Wire Wire Line
+	3200 1050 3200 1000
+Wire Wire Line
+	2800 1400 3450 1400
 $EndSCHEMATC

Commit message: * placed components on PCB and started positioning
Parts:
- C1: renamed from C?; value C -> 1u; footprint (none) -> Capacitors_SMD:C_0805
- C2, C3, C4: renamed from C?; footprint (none) -> Capacitors_SMD:C_0805
- J1, J2: renamed from J?; footprint (none) -> SquantorConnectors:Header-2.54-1X06-H0.8
- R1, R2, R3: renamed from R?; footprint (none) -> Resistors_SMD:R_0805
- RV1: renamed from RV?; footprint (none) -> Potentiometers:Potentiometer_Bourns_3296W_3-8Zoll_Inline_ScrewUp
- U1: renamed from U?; footprint (none) -> SquantorIC:SquantorIC-SO08
Connections:
- wire segments 19 -> 22
Other:
- moved on the sheet: C1, C2, C3, C4, R1, R2, R3, RV1, U1

Commit message: * Some more layouting of the REF50XX module
Parts:
- RV1: symbol POT -> POT-RESCUE-REF50XX_module
Changed lines of the file:
@@
 EESchema Schematic File Version 2
+LIBS:REF50XX_module-rescue
 LIBS:power
 LIBS:device
@@
 LIBS:SquantorConnectors
 LIBS:SquantorTexasInstruments
+LIBS:REF50XX_module-cache
 EELAYER 25 0
 EELAYER END
@@
 $EndComp
 $Comp
-L POT RV1
+L POT-RESCUE-REF50XX_module RV1
 U 1 1 585464D5
 P 3500 2100

Commit message: * redid partially REF5040 reference board
Parts:
- removed J1, J2: PINS_1X6, SquantorConnectors:Header-2.54-1X06-H0.8, symbol PINS_1X6
- removed RV1: 10k, Potentiometers:Potentiometer_Bourns_3296W_3-8Zoll_Inline_ScrewUp, symbol POT-RESCUE-REF50XX_module
- added C5: 4.7u, SquantorRcl:C025-055X046, symbol C
- added J1, J2: PINS_1X8, SquantorConnectors:Header-0254-1X08-H010, symbol PINS_1X8
- added R4: 0, Resistors_SMD:R_0603, symbol R
- added R5: 0, Resistors_SMD:R_0805, symbol R
- added RV1: 10k, SquantorRcl:POT_SMD_44W, symbol POT
Connections:
- net labels added: Heater, HeaterGround, RefTemp, Sense, Vin, Vref
- wire segments 22 -> 49
Other:
- moved on the sheet: C3, C4, R3
