File: hardware/bypass_capacitor_tester/bypass_capacitor_tester.kicad_pcb (KiCad board)
At the start: 2 copper layers, 2 parts

Commit message: started layout
Parts:
- added C1: DUT, SquantorRcl:C_0805+0603, F.Cu at (190.0, 73.0)
- added FB1: Ferrite_Bead, SquantorRcl:C_0805+0603, F.Cu at (195.0, 73.0)
- added J1: Coax, SquantorConnectors:Conn_BNC_RightAngle_TH, B.Cu at (198.0, 92.0)
- added J2: Coax, SquantorConnectors:Conn_BNC_RightAngle_TH, B.Cu at (176.0, 92.0)
- added J3: Coax, SquantorConnectors:Conn_BNC_RightAngle_TH, B.Cu at (176.0, 76.0)
- added J4: Conn_01x02, Connector_PinHeader_2.54mm:PinHeader_1x02_P2.54mm_Horizontal, B.Cu at (195.0, 80.0)
- added Q1: MMBT2369AL, SquantorIC:SOT23-3, F.Cu at (188.0, 86.3)
- added R1: 50, SquantorRcl:R_0805+0603, F.Cu at (187.0, 92.8)
- added R2: 560, SquantorRcl:R_0805+0603, F.Cu at (187.0, 89.7)
- added R3: 100, SquantorRcl:R_0805+0603, F.Cu at (188.0, 82.9)
- added R4: 50, SquantorRcl:R_0805+0603, F.Cu at (185.6, 76.7)
- N1: moved to B.Cu
- N2: value 20190704 -> 20191105; moved to B.Cu
- moved N1 48.7 mm to (188.5, 74.0), turned to 180 degrees
- moved N2 47.4 mm to (188.0, 78.0)
Routing:
- net /A_WAVEFORM: track 0.00 -> 13.4 mm
- net Net-(Q1-Pad1): track 0.00 -> 1.65 mm
- net Net-(Q1-Pad3): track 0.00 -> 1.62 mm
- net GND: vias 0 -> 45
- added copper zone on B.Cu, net GND
- added copper zone on F.Cu, net GND
Other:
- board outline added: 40 x 34 mm
