File: electronics/dslogic_base/dslogic_base.kicad_sch (KiCad schematic)
At the start: 3 parts, among them J1 Conn_02x23_Odd_Even

Commit message: completed schematic, board layout and updated readme
Parts:
- added J2, J3: Conn_02x08_Odd_Even, Connector_PinHeader_1.27mm:PinHeader_2x08_P1.27mm_Vertical, symbol Connector_Generic:Conn_02x08_Odd_Even
- J1: footprint Connector_PinHeader_1.27mm:PinHeader_2x23_P1.27mm_Horizontal -> Connector_PinHeader_1.27mm:PinHeader_2x22_P1.27mm_Vertical
Connections:
- net GND: now also J1.1 (Pin_1), J1.11 (Pin_11), J1.13 (Pin_13), J1.15 (Pin_15), J1.17 (Pin_17), J1.21 (Pin_21), J1.23 (Pin_23), J1.25 (Pin_25), J1.27 (Pin_27), J1.3 (Pin_3), J1.31 (Pin_31), J1.33 (Pin_33), J1.35 (Pin_35), J1.37 (Pin_37), J1.41 (Pin_41), J1.43 (Pin_43), J1.45 (Pin_45), J1.5 (Pin_5), J1.7 (Pin_7), J2.10 (Pin_10), J2.12 (Pin_12), J2.14 (Pin_14), J2.16 (Pin_16), J2.2 (Pin_2), J2.4 (Pin_4), J2.6 (Pin_6), J2.8 (Pin_8), J3.10 (Pin_10), J3.12 (Pin_12), J3.14 (Pin_14), J3.16 (Pin_16), J3.2 (Pin_2), J3.4 (Pin_4), J3.6 (Pin_6), J3.8 (Pin_8); no longer J1.10 (Pin_10), J1.12 (Pin_12), J1.14 (Pin_14), J1.16 (Pin_16), J1.18 (Pin_18), J1.2 (Pin_2), J1.20 (Pin_20), J1.22 (Pin_22), J1.24 (Pin_24), J1.26 (Pin_26), J1.28 (Pin_28), J1.30 (Pin_30), J1.32 (Pin_32), J1.34 (Pin_34), J1.36 (Pin_36), J1.38 (Pin_38), J1.4 (Pin_4), J1.40 (Pin_40), J1.42 (Pin_42), J1.44 (Pin_44), J1.46 (Pin_46), J1.6 (Pin_6), J1.8 (Pin_8)
- new net CH00: J1.2 (Pin_2), J2.1 (Pin_1)
- new net CH01: J1.4 (Pin_4), J2.3 (Pin_3)
- new net CH02: J1.6 (Pin_6), J2.5 (Pin_5)
- new net CH03: J1.8 (Pin_8), J2.7 (Pin_7)
- new net CH04: J1.12 (Pin_12), J2.9 (Pin_9)
- new net CH05: J1.14 (Pin_14), J2.11 (Pin_11)
- new net CH06: J1.16 (Pin_16), J2.13 (Pin_13)
- new net CH07: J1.18 (Pin_18), J2.15 (Pin_15)
- new net CH08: J1.22 (Pin_22), J3.1 (Pin_1)
- new net CH09: J1.24 (Pin_24), J3.3 (Pin_3)
- new net CH10: J1.26 (Pin_26), J3.5 (Pin_5)
- new net CH11: J1.28 (Pin_28), J3.7 (Pin_7)
- new net CH12: J1.32 (Pin_32), J3.9 (Pin_9)
- new net CH13: J1.34 (Pin_34), J3.11 (Pin_11)
- new net CH14: J1.36 (Pin_36), J3.13 (Pin_13)
- new net CH15: J1.38 (Pin_38), J3.15 (Pin_15)
- no-connect marks 0 -> 11

Commit message: updated versionnumber and reviewed
Parts:
- N1: value 20220923 -> 20221009
Other:
- note added: "Connections"
- moved on the sheet: J3
