File: electronics/dslogic_probe_4/dslogic_probe_4.kicad_pcb (KiCad board)
At the start: 2 copper layers, 11.3 x 6 mm, 16 parts, among them J1 Conn_02x04_Odd_Even, J2 Conn_02x04_Odd_Even

Commit message: reviewd 4 bit logic probe circuit
Parts:
- N1: value 20220506 -> 20221009
Changed lines of the file:
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@@
   (net 4 "Net-(C2-Pad2)")
   (net 5 "Net-(C3-Pad2)")
-  (net 6 "Net-(J2-Pad3)")
+  (net 6 "Net-(C3-Pad1)")
   (net 7 "Net-(C4-Pad2)")
   (net 8 "/GND")
-  (net 9 "Net-(J2-Pad1)")
+  (net 9 "Net-(C4-Pad1)")
   (net 10 "Net-(J1-Pad2)")
   (net 11 "Net-(J1-Pad4)")
@@
     (fp_line (start 0.5 -0.25) (end 0.5 0.25) (layer "F.Fab") (width 0.1))
     (pad "1" smd rect (at -0.55 0) (size 0.6 0.6) (layers "F.Cu" "F.Paste" "F.Mask")
-      (net 6 "Net-(J2-Pad3)") (pintype "passive"))
+      (net 6 "Net-(C3-Pad1)") (pintype "passive"))
     (pad "2" smd rect (at 0.55 0) (size 0.6 0.6) (layers "F.Cu" "F.Paste" "F.Mask")
       (net 5 "Net-(C3-Pad2)") (pintype "passive"))
@@
     (fp_line (start -0.5 0.25) (end -0.5 -0.25) (layer "F.Fab") (width 0.1))
     (pad "1" smd rect (at -0.55 0) (size 0.6 0.6) (layers "F.Cu" "F.Paste" "F.Mask")
-      (net 9 "Net-(J2-Pad1)") (pintype "passive"))
+      (net 9 "Net-(C4-Pad1)") (pintype "passive"))
     (pad "2" smd rect (at 0.55 0) (size 0.6 0.6) (layers "F.Cu" "F.Paste" "F.Mask")
       (net 7 "Net-(C4-Pad2)") (pintype "passive"))
@@
       (effects (font (size 1 1) (thickness 0.15)) (justify mirror))
     )
-    (fp_text value "20220506" (at 0.8 0.1 90) (layer "B.SilkS")
+    (fp_text value "20221009" (at 0.8 0.1 90) (layer "B.SilkS")
       (effects (font (size 0.8 0.8) (thickness 0.15)) (justify mirror))
     )
@@
     (fp_line (start 2.7 0.3) (end 2.7 -2.5) (layer "F.CrtYd") (width 0.05))
     (pad "1" smd roundrect (at -1.905 -1.1 90) (size 0.8 2) (layers "F.Cu" "F.Paste" "F.Mask") (roundrect_rratio 0.25)
-      (net 9 "Net-(J2-Pad1)") (pinfunction "Pin_1") (pintype "passive"))
+      (net 9 "Net-(C4-Pad1)") (pinfunction "Pin_1") (pintype "passive"))
     (pad "2" smd rect (at -1.905 -1.1 90) (size 0.8 2) (layers "B.Cu" "B.Paste" "B.Mask")
       (net 8 "/GND") (pinfunction "Pin_2") (pintype "passive") (zone_connect 2))
     (pad "3" smd rect (at -0.635 -1.1 90) (size 0.8 2) (layers "F.Cu" "F.Paste" "F.Mask")
-      (net 6 "Net-(J2-Pad3)") (pinfunction "Pin_3") (pintype "passive"))
+      (net 6 "Net-(C3-Pad1)") (pinfunction "Pin_3") (pintype "passive"))
     (pad "4" smd rect (at -0.635 -1.1 90) (size 0.8 2) (layers "B.Cu" "B.Paste" "B.Mask")
       (net 8 "/GND") (pinfunction "Pin_4") (pintype "passive") (zone_connect 2))
@@
     (fp_line (start -0.5 -0.25) (end -0.5 0.25) (layer "B.Fab") (width 0.1))
     (pad "1" smd rect (at -0.55 0) (size 0.6 0.6) (layers "B.Cu" "B.Paste" "B.Mask")
-      (net 6 "Net-(J2-Pad3)") (pintype "passive"))
+      (net 6 "Net-(C3-Pad1)") (pintype "passive"))
     (pad "2" smd rect (at 0.55 0) (size 0.6 0.6) (layers "B.Cu" "B.Paste" "B.Mask")
       (net 5 "Net-(C3-Pad2)") (pintype "passive"))
@@
     (fp_line (start 0.5 -0.25) (end -0.5 -0.25) (layer "B.Fab") (width 0.1))
     (pad "1" smd rect (at -0.55 0) (size 0.6 0.6) (layers "B.Cu" "B.Paste" "B.Mask")
-      (net 9 "Net-(J2-Pad1)") (pintype "passive"))
+      (net 9 "Net-(C4-Pad1)") (pintype "passive"))
     (pad "2" smd rect (at 0.55 0) (size 0.6 0.6) (layers "B.Cu" "B.Paste" "B.Mask")
       (net 7 "Net-(C4-Pad2)") (pintype "passive"))

Commit message: minor changes
Parts:
- removed N2: OHWLOGO, Symbol:OSHW-Symbol_6.7x6mm_SilkScreen
Other:
- board size 11.3 x 6 mm -> 11.3 x 6.4 mm
