File: electronics/oscillator_variant_1/oscillator_variant_1.kicad_pcb (KiCad board)
At the start: 2 copper layers, 42.5 x 46.2 mm, 51 parts, among them J1 module_2x15_left_input, J2 module_2x15_right_input, J3 Coax, Q1 BC817, U1 TL081, U2 LME49720, U3 TL082, U4 TL431

Commit message: reviewed
Parts:
- N1: value 20220501 -> 20220507
Changed lines of the file:
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@@
       (effects (font (size 1 1) (thickness 0.15)) (justify mirror))
     )
-    (fp_text value "20220501" (at 0.8 0.1) (layer "B.SilkS")
+    (fp_text value "20220507" (at 0.8 0.1) (layer "B.SilkS")
       (effects (font (size 0.8 0.8) (thickness 0.15)) (justify mirror))
     )

Commit message: fixed aisler warnings/errors
Parts:
- C4, C5, C6: footprint SquantorRcl:C-025_050-050X100-0805-3516-film -> SquantorRcl:C-050-050X100-0805-3516-film
- N1: value 20220507 -> 20220530
