File: electronics/notch_filter/notch_filter.kicad_pcb (KiCad board)
At the start: 2 copper layers, 42.4 x 46.2 mm, 39 parts, among them J1 Conn_01x03, J2 Conn_01x03, J3 Output, J4 In, J5 module_2x15_left_input, J6 module_2x15_right_input, U1 opamp_single_8pin

Commit message: removed labels and minor optimisations
Parts:
- removed N3: A:, SquantorLabels:Label_Note_medium
- removed N4: B:, SquantorLabels:Label_Note_medium
- removed N5: C:, SquantorLabels:Label_Note_medium
- removed N6: D:, SquantorLabels:Label_Note_medium
- removed N7: E:, SquantorLabels:Label_Note_medium
- removed N8: Hz:, SquantorLabels:Label_Note_medium
- N1: value 20230530 -> 20230717
